File: openlst-hw.kicad_sch (KiCad schematic)
At the start: 69 parts, among them J3 Conn_02x10_Odd_Even, J6 ANT, U2 CC1110, U4 ASFL1-27.000MHZ, U5 MIC803, U6 PE4250, U7 RFFM6406, U8 SF2446E

Commit message: fixed TR components
Parts:
- L2: SupplierPN 240-2407-2-ND -> 240-2407-1-ND
- TP1, TP2: SupplierPN 2019-RCUCTETR-ND -> 2019-RCUCTECT-ND
Changed lines of the file:
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@@
       (effects (font (size 1.524 1.524)) hide)
     )
-    (property "SupplierPN" "240-2407-2-ND" (at 288.29 82.55 90)
+    (property "SupplierPN" "240-2407-1-ND" (at 288.29 82.55 90)
       (effects (font (size 1.524 1.524)) hide)
     )
@@
       (effects (font (size 1.27 1.27)) hide)
     )
-    (property "SupplierPN" "2019-RCUCTETR-ND" (at 60.96 168.91 0)
+    (property "SupplierPN" "2019-RCUCTECT-ND" (at 60.96 168.91 0)
       (effects (font (size 1.27 1.27)) hide)
     )
@@
       (effects (font (size 1.27 1.27)) hide)
     )
-    (property "SupplierPN" "2019-RCUCTETR-ND" (at 64.77 166.37 0)
-      (effects (font (size 1.27 1.27)) hide)
-    )
+    (property "SupplierPN" "2019-RCUCTECT-ND" (at 64.77 166.37 0)
+      (effects (font (size 1.27 1.27)) hide)
+    )

Commit message: changed MMCXV-J-P-HF-ST-TH1 to a digikey part
Parts:
- J6: Supplier Samtec -> Digikey; SupplierPN MMCXV-J-P-HF-ST-TH1 -> SAM11508-ND
Changed lines of the file:
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@@
       (effects (font (size 1.27 1.27)) hide)
     )
-    (property "Supplier" "Samtec" (at 302.26 129.54 0)
+    (property "Supplier" "Digikey" (at 302.26 129.54 0)
       (effects (font (size 1.27 1.27)) hide)
     )
-    (property "SupplierPN" "MMCXV-J-P-HF-ST-TH1" (at 302.26 129.54 0)
+    (property "SupplierPN" "SAM11508-ND" (at 302.26 129.54 0)
       (effects (font (size 1.27 1.27)) hide)
     )
